File: pcb/userport_connector/userport_connector.kicad_pcb (KiCad board)
At the start: 2 copper layers, 30.9 x 52.7 mm, 6 parts, among them J1 PET User Port, J2 Raspberry_Pi_2_3, U1 74LVC245

Commit message: fixed board problem
Connections:
- J2 pad 27: D0 -> Net-(J2-Pad27)
- J2 pad 28: Net-(J2-Pad28) -> D2
Routing:
- net D0: track 18.6 -> 4.97 mm
- net GND: track 126.3 -> 118.0 mm
- net D2: track 0.00 -> 7.24 mm
- net D3: track 15.9 -> 12.6 mm
- net D6: track 12.5 -> 15.8 mm
- net +3V3: track 52.9 -> 54.6 mm
